File: balenaFin v1.1 HAT Template/KiCAD/FIN_HAT_Template.kicad_pcb (KiCad board)
At the start: 2 copper layers, 90 x 73 mm, 6 parts, among them J1 Raspberry_Pi_2_3, J2 POE_Header, J3 Co-Processor_Header, J4 USB_Header

Commit message: Solved the 3D models issue and converted the male pin headers to female sokets
Parts:
- J1: footprint FIN HAT Template:PinHeader_2x20_P2.54mm_Vertical -> FIN HAT Template:PinSocket_2x20_P2.54mm_Vertical
- J2: footprint FIN HAT Template:PinHeader_2x02_P2.54mm_Vertical -> FIN HAT Template:PinSocket_2x02_P2.54mm_Vertical
- J3: footprint FIN HAT Template:PinHeader_2x09_P2.54mm_Vertical -> FIN HAT Template:PinSocket_2x09_P2.54mm_Vertical
- J4: footprint FIN HAT Template:PinHeader_1x04_P2.54mm_Vertical -> FIN HAT Template:PinSocket_1x04_P2.54mm_Vertical

Commit message: Fixed the orientaion of the POE header
Parts:
- turned J2 to 270 degrees
Changed lines of the file:
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@@
     (descr "Through hole straight socket strip, 1x04, 2.54mm pitch, single row (from Kicad 4.0.7), script generated")
     (tags "Through hole socket strip THT 1x04 2.54mm single row")
-    (fp_text reference J4 (at 0 6.58 90) (layer B.SilkS)
+    (fp_text reference J4 (at 0 6.58 180) (layer B.SilkS)
       (effects (font (size 1 1) (thickness 0.15)) (justify mirror))
     )
@@
   )
   (module "FIN HAT Template:PinSocket_2x02_P2.54mm_Vertical" (layer B.Cu)
-    (at 113.01 71.85)
+    (at 113.01 71.85 270)
     (descr "Through hole straight socket strip, 2x02, 2.54mm pitch, double cols (from Kicad 4.0.7), script generated")
     (tags "Through hole socket strip THT 2x02 2.54mm double row")
-    (fp_text reference J2 (at 0 4.04) (layer B.SilkS)
+    (fp_text reference J2 (at 0 4.04 180) (layer B.SilkS)
       (effects (font (size 1 1) (thickness 0.15)) (justify mirror))
     )
-    (fp_text value POE_Header (at 0 -4.04) (layer B.Fab)
+    (fp_text value POE_Header (at 0 -4.04 90) (layer B.Fab)
       (effects (font (size 1 1) (thickness 0.15)) (justify mirror))
     )
-    (fp_text user %R (at 0 0 -90) (layer B.Fab)
+    (fp_text user %R (at 0 0 180) (layer B.Fab)
       (effects (font (size 1 1) (thickness 0.15)) (justify mirror))
     )
@@
     (fp_line (start 3.03 -3.03) (end -3.07 -3.03) (layer B.CrtYd) (width 0.05))
     (fp_line (start -3.07 -3.03) (end -3.07 3.07) (layer B.CrtYd) (width 0.05))
-    (pad 4 thru_hole oval (at -1.27 -1.27) (size 1.7 1.7) (drill 1) (layers *.Cu *.Mask)
+    (pad 4 thru_hole oval (at -1.27 -1.27 270) (size 1.7 1.7) (drill 1) (layers *.Cu *.Mask)
       (net 37 "Net-(J2-Pad4)"))
-    (pad 3 thru_hole oval (at 1.27 -1.27) (size 1.7 1.7) (drill 1) (layers *.Cu *.Mask)
+    (pad 3 thru_hole oval (at 1.27 -1.27 270) (size 1.7 1.7) (drill 1) (layers *.Cu *.Mask)
       (net 36 "Net-(J2-Pad3)"))
-    (pad 2 thru_hole oval (at -1.27 1.27) (size 1.7 1.7) (drill 1) (layers *.Cu *.Mask)
+    (pad 2 thru_hole oval (at -1.27 1.27 270) (size 1.7 1.7) (drill 1) (layers *.Cu *.Mask)
       (net 35 "Net-(J2-Pad2)"))
-    (pad 1 thru_hole rect (at 1.27 1.27) (size 1.7 1.7) (drill 1) (layers *.Cu *.Mask)
+    (pad 1 thru_hole rect (at 1.27 1.27 270) (size 1.7 1.7) (drill 1) (layers *.Cu *.Mask)
       (net 34 "Net-(J2-Pad1)"))
     (model ${KISYS3DMOD}/Connector_PinSocket_2.54mm.3dshapes/PinSocket_2x02_P2.54mm_Vertical.wrl
