File: balenaFin v1.1 HAT Template/KiCAD/FIN_HAT_Template.sch (KiCad schematic (older format))
At the start: 6 parts, among them J1 Raspberry_Pi_2_3, J2 Conn_02x02_Top_Bottom, J3 Conn_02x09_Top_Bottom, J4 Conn_01x04_Female

Commit message: Created a lib for our schematic symbols
Parts:
- removed J2: Conn_02x02_Top_Bottom, Connector_PinHeader_2.54mm:PinHeader_2x02_P2.54mm_Vertical, symbol Connector_Generic:Conn_02x02_Top_Bottom
- removed J3: Conn_02x09_Top_Bottom, Connector_PinHeader_2.54mm:PinHeader_2x09_P2.54mm_Vertical, symbol Connector_Generic:Conn_02x09_Top_Bottom
- removed J4: Conn_01x04_Female, Connector_PinHeader_2.54mm:PinHeader_1x04_P2.54mm_Vertical, symbol Connector:Conn_01x04_Female
- added J2: POE_Header, Connector_PinHeader_2.54mm:PinHeader_2x02_P2.54mm_Vertical, symbol FIN_HAT_TEMPLATE:POE_Header
- added J3: Co-Processor_Header, Connector_PinHeader_2.54mm:PinHeader_2x09_P2.54mm_Vertical, symbol FIN_HAT_TEMPLATE:Co-Processor_Header
- added J4: USB_Header, Connector_PinHeader_2.54mm:PinHeader_1x04_P2.54mm_Vertical, symbol FIN_HAT_TEMPLATE:USB_Header
Connections:
- net +5V: now also J4.1 (5V)
- net GND: now also J3.17 (GND), J4.4 (GND)
- no-connect marks 56 -> 53
Changed lines of the file:
@@
 $EndDescr
 $Comp
-L power:GND #PWR0101
+L power:GND #PWR02
 U 1 1 5F07D099
 P 3450 5300
-F 0 "#PWR0101" H 3450 5050 50  0001 C CNN
+F 0 "#PWR02" H 3450 5050 50  0001 C CNN
 F 1 "GND" H 3455 5127 50  0000 C CNN
 F 2 "" H 3450 5300 50  0001 C CNN
@@
 	3750 2200 3750 2500
 $Comp
-L power:+3.3V #PWR0102
+L power:+3.3V #PWR03
 U 1 1 5F07F1C6
 P 3750 2000
-F 0 "#PWR0102" H 3750 1850 50  0001 C CNN
+F 0 "#PWR03" H 3750 1850 50  0001 C CNN
 F 1 "+3.3V" H 3765 2173 50  0000 C CNN
 F 2 "" H 3750 2000 50  0001 C CNN
@@
 $EndComp
 $Comp
-L power:+5V #PWR0103
+L power:+5V #PWR01
 U 1 1 5F07F8B1
 P 3350 2000
-F 0 "#PWR0103" H 3350 1850 50  0001 C CNN
+F 0 "#PWR01" H 3350 1850 50  0001 C CNN
 F 1 "+5V" H 3365 2173 50  0000 C CNN
 F 2 "" H 3350 2000 50  0001 C CNN
@@
 	3750 2000 3750 2200
 Connection ~ 3750 2200
-$Comp
-L Connector:Conn_01x04_Female J4
-U 1 1 5F0810CB
-P 10100 2300
-F 0 "J4" H 10128 2276 50  0000 L CNN
-F 1 "Conn_01x04_Female" H 10128 2185 50  0000 L CNN
-F 2 "Connector_PinHeader_2.54mm:PinHeader_1x04_P2.54mm_Vertical" H 10100 2300 50  0001 C CNN
-F 3 "~" H 10100 2300 50  0001 C CNN
-	1    10100 2300
-	1    0    0    -1
-$EndComp
-$Comp
-L Connector_Generic:Conn_02x09_Top_Bottom J3
-U 1 1 5F082D48
-P 10000 4450
-F 0 "J3" H 10050 5067 50  0000 C CNN
-F 1 "Conn_02x09_Top_Bottom" H 10050 4976 50  0000 C CNN
-F 2 "Connector_PinHeader_2.54mm:PinHeader_2x09_P2.54mm_Vertical" H 10000 4450 50  0001 C CNN
-F 3 "~" H 10000 4450 50  0001 C CNN
-	1    10000 4450
-	1    0    0    -1
-$EndComp
-$Comp
-L Connector_Generic:Conn_02x02_Top_Bottom J2
-U 1 1 5F084777
-P 8100 2250
-F 0 "J2" H 8150 2467 50  0000 C CNN
-F 1 "Conn_02x02_Top_Bottom" H 8150 2376 50  0000 C CNN
-F 2 "Connector_PinHeader_2.54mm:PinHeader_2x02_P2.54mm_Vertical" H 8100 2250 50  0001 C CNN
-F 3 "~" H 8100 2250 50  0001 C CNN
-	1    8100 2250
-	1    0    0    -1
-$EndComp
 $Comp
 L Mechanical:MountingHole_Pad H2
@@
 Text Notes 7900 2550 0    50   ~ 0
 POE Header
-Text Notes 9800 2750 0    50   ~ 0
+Text Notes 10100 2700 0    50   ~ 0
 USB Header
 Text Notes 4000 5100 0    50   ~ 0
@@
 NoConn ~ 2750 4400
 NoConn ~ 2750 4500
-NoConn ~ 7900 2250
-NoConn ~ 7900 2350
-NoConn ~ 8400 2250
-NoConn ~ 8400 2350
+NoConn ~ 7700 2300
+NoConn ~ 7700 2400
+NoConn ~ 8600 2300
+NoConn ~ 8600 2400
 NoConn ~ 8400 1400
 NoConn ~ 9550 1400
-NoConn ~ 9900 2200
 NoConn ~ 9900 2300
 NoConn ~ 9900 2400
-NoConn ~ 9900 2500
-NoConn ~ 9800 4050
-NoConn ~ 10300 4050
-NoConn ~ 10300 4150
-NoConn ~ 9800 4150
-NoConn ~ 9800 4250
-NoConn ~ 9800 4350
-NoConn ~ 9800 4450
-NoConn ~ 9800 4550
-NoConn ~ 9800 4650
-NoConn ~ 9800 4750
-NoConn ~ 9800 4850
-NoConn ~ 10300 4850
-NoConn ~ 10300 4750
-NoConn ~ 10300 4650
-NoConn ~ 10300 4550
-NoConn ~ 10300 4450
-NoConn ~ 10300 4350
-NoConn ~ 10300 4250
-$Comp
-L power:PWR_FLAG #FLG0101
+NoConn ~ 9500 4050
+NoConn ~ 10600 4150
+NoConn ~ 9500 4150
+NoConn ~ 9500 4250
+NoConn ~ 9500 4350
+NoConn ~ 9500 4450
+NoConn ~ 9500 4550
+NoConn ~ 9500 4650
+NoConn ~ 9500 4750
+NoConn ~ 10600 4850
+NoConn ~ 10600 4750
+NoConn ~ 10600 4650
+NoConn ~ 10600 4550
+NoConn ~ 10600 4450
+NoConn ~ 10600 4350
+NoConn ~ 10600 4250
+$Comp
+L power:PWR_FLAG #FLG01
 U 1 1 5F0A5218
 P 5600 1100
-F 0 "#FLG0101" H 5600 1175 50  0001 C CNN
+F 0 "#FLG01" H 5600 1175 50  0001 C CNN
 F 1 "PWR_FLAG" H 5600 1273 50  0000 C CNN
 F 2 "" H 5600 1100 50  0001 C CNN
@@
 $EndComp
 $Comp
-L power:PWR_FLAG #FLG0102
+L power:PWR_FLAG #FLG02
 U 1 1 5F0A5889
 P 6150 1100
-F 0 "#FLG0102" H 6150 1175 50  0001 C CNN
+F 0 "#FLG02" H 6150 1175 50  0001 C CNN
 F 1 "PWR_FLAG" H 6150 1273 50  0000 C CNN
 F 2 "" H 6150 1100 50  0001 C CNN
@@
 $EndComp
 $Comp
-L power:+3.3V #PWR0104
+L power:+3.3V #PWR04
 U 1 1 5F0A5D68
 P 5600 1300
-F 0 "#PWR0104" H 5600 1150 50  0001 C CNN
+F 0 "#PWR04" H 5600 1150 50  0001 C CNN
 F 1 "+3.3V" H 5615 1473 50  0000 C CNN
 F 2 "" H 5600 1300 50  0001 C CNN
@@
 $EndComp
 $Comp
-L power:+5V #PWR0105
+L power:+5V #PWR05
 U 1 1 5F0A64A2
 P 6150 1300
-F 0 "#PWR0105" H 6150 1150 50  0001 C CNN
+F 0 "#PWR05" H 6150 1150 50  0001 C CNN
 F 1 "+5V" H 6165 1473 50  0000 C CNN
 F 2 "" H 6150 1300 50  0001 C CNN
@@
 $EndComp
 $Comp
-L power:PWR_FLAG #FLG0103
+L power:PWR_FLAG #FLG03
 U 1 1 5F0A7111
 P 6700 1100
-F 0 "#FLG0103" H 6700 1175 50  0001 C CNN
+F 0 "#FLG03" H 6700 1175 50  0001 C CNN
 F 1 "PWR_FLAG" H 6700 1273 50  0000 C CNN
 F 2 "" H 6700 1100 50  0001 C CNN
@@
 $EndComp
 $Comp
-L power:GND #PWR0106
+L power:GND #PWR06
 U 1 1 5F0A74E3
 P 6700 1300
-F 0 "#PWR0106" H 6700 1050 50  0001 C CNN
+F 0 "#PWR06" H 6700 1050 50  0001 C CNN
 F 1 "GND" H 6705 1127 50  0000 C CNN
 F 2 "" H 6700 1300 50  0001 C CNN
@@
 Wire Wire Line
 	6700 1300 6700 1100
+$Comp
+L FIN_HAT_TEMPLATE:Co-Processor_Header J3
+U 1 1 5F1CE898
+P 9700 4050
+F 0 "J3" H 10050 4275 50  0000 C CNN
+F 1 "Co-Processor_Header" H 10050 4184 50  0000 C CNN
+F 2 "Connector_PinHeader_2.54mm:PinHeader_2x09_P2.54mm_Vertical" H 9700 3650 50  0001 C CNN
+F 3 "~" H 9700 3650 50  0001 C CNN
+	1    9700 4050
+	1    0    0    -1
+$EndComp
+NoConn ~ 10600 4050
+$Comp
+L power:GND #PWR07
+U 1 1 5F1D21C3
+P 9400 5000
+F 0 "#PWR07" H 9400 4750 50  0001 C CNN
+F 1 "GND" H 9405 4827 50  0000 C CNN
+F 2 "" H 9400 5000 50  0001 C CNN
+F 3 "" H 9400 5000 50  0001 C CNN
+	1    9400 5000
+	1    0    0    -1
+$EndComp
+Wire Wire Line
+	9400 5000 9400 4850
+Wire Wire Line
+	9400 4850 9500 4850
+$Comp
+L FIN_HAT_TEMPLATE:POE_Header J2
+U 1 1 5F1D361B
+P 7900 2300
+F 0 "J2" H 8150 2525 50  0000 C CNN
+F 1 "POE_Header" H 8150 2434 50  0000 C CNN
+F 2 "Connector_PinHeader_2.54mm:PinHeader_2x02_P2.54mm_Vertical" H 7900 2300 50  0001 C CNN
+F 3 "~" H 7900 2300 50  0001 C CNN
+	1    7900 2300
+	1    0    0    -1
+$EndComp
+$Comp
+L FIN_HAT_TEMPLATE:USB_Header J4
+U 1 1 5F1D6217
+P 10100 2300
+F 0 "J4" H 10328 2301 50  0000 L CNN
+F 1 "USB_Header" H 10328 2210 50  0000 L CNN
+F 2 "Connector_PinHeader_2.54mm:PinHeader_1x04_P2.54mm_Vertical" H 10100 2300 50  0001 C CNN
+F 3 "~" H 10100 2300 50  0001 C CNN
+	1    10100 2300
+	1    0    0    -1
+$EndComp
+$Comp
+L power:GND #PWR09
+U 1 1 5F1D6ACD
+P 9800 2600
+F 0 "#PWR09" H 9800 2350 50  0001 C CNN
+F 1 "GND" H 9805 2427 50  0000 C CNN
+F 2 "" H 9800 2600 50  0001 C CNN
+F 3 "" H 9800 2600 50  0001 C CNN
+	1    9800 2600
+	1    0    0    -1
+$EndComp
+$Comp
+L power:+5V #PWR08
+U 1 1 5F1D74CB
+P 9800 2100
+F 0 "#PWR08" H 9800 1950 50  0001 C CNN
+F 1 "+5V" H 9815 2273 50  0000 C CNN
+F 2 "" H 9800 2100 50  0001 C CNN
+F 3 "" H 9800 2100 50  0001 C CNN
+	1    9800 2100
+	1    0    0    -1
+$EndComp
+Wire Wire Line
+	9900 2200 9800 2200
+Wire Wire Line
+	9800 2200 9800 2100
+Wire Wire Line
+	9900 2500 9800 2500
+Wire Wire Line
+	9800 2500 9800 2600
 $EndSCHEMATC

Commit message: Created footrpints lib - Fixed the mirrored footprints issue - Added the dimenions
Parts:
- J1: footprint Connector_PinHeader_2.54mm:PinHeader_2x20_P2.54mm_Vertical -> FIN HAT Template:PinHeader_2x20_P2.54mm_Vertical
- J2: footprint Connector_PinHeader_2.54mm:PinHeader_2x02_P2.54mm_Vertical -> FIN HAT Template:PinHeader_2x02_P2.54mm_Vertical
- J3: footprint Connector_PinHeader_2.54mm:PinHeader_2x09_P2.54mm_Vertical -> FIN HAT Template:PinHeader_2x09_P2.54mm_Vertical
- J4: footprint Connector_PinHeader_2.54mm:PinHeader_1x04_P2.54mm_Vertical -> FIN HAT Template:PinHeader_1x04_P2.54mm_Vertical
Changed lines of the file:
@@
 F 0 "J1" H 2550 5200 50  0000 C CNN
 F 1 "Raspberry_Pi_2_3" H 2850 5100 50  0000 C CNN
-F 2 "Connector_PinHeader_2.54mm:PinHeader_2x20_P2.54mm_Vertical" H 3550 3800 50  0001 C CNN
+F 2 "FIN HAT Template:PinHeader_2x20_P2.54mm_Vertical" H 3550 3800 50  0001 C CNN
 F 3 "https://www.raspberrypi.org/documentation/hardware/raspberrypi/schematics/rpi_SCH_3bplus_1p0_reduced.pdf" H 3550 3800 50  0001 C CNN
 	1    3550 3800
@@
 F 0 "J3" H 10050 4275 50  0000 C CNN
 F 1 "Co-Processor_Header" H 10050 4184 50  0000 C CNN
-F 2 "Connector_PinHeader_2.54mm:PinHeader_2x09_P2.54mm_Vertical" H 9700 3650 50  0001 C CNN
+F 2 "FIN HAT Template:PinHeader_2x09_P2.54mm_Vertical" H 9700 3650 50  0001 C CNN
 F 3 "~" H 9700 3650 50  0001 C CNN
 	1    9700 4050
@@
 F 0 "J2" H 8150 2525 50  0000 C CNN
 F 1 "POE_Header" H 8150 2434 50  0000 C CNN
-F 2 "Connector_PinHeader_2.54mm:PinHeader_2x02_P2.54mm_Vertical" H 7900 2300 50  0001 C CNN
+F 2 "FIN HAT Template:PinHeader_2x02_P2.54mm_Vertical" H 7900 2300 50  0001 C CNN
 F 3 "~" H 7900 2300 50  0001 C CNN
 	1    7900 2300
@@
 F 0 "J4" H 10328 2301 50  0000 L CNN
 F 1 "USB_Header" H 10328 2210 50  0000 L CNN
-F 2 "Connector_PinHeader_2.54mm:PinHeader_1x04_P2.54mm_Vertical" H 10100 2300 50  0001 C CNN
+F 2 "FIN HAT Template:PinHeader_1x04_P2.54mm_Vertical" H 10100 2300 50  0001 C CNN
 F 3 "~" H 10100 2300 50  0001 C CNN
 	1    10100 2300

Commit message: Solved the 3D models issue and converted the male pin headers to female sokets
Parts:
- removed J1: Raspberry_Pi_2_3, FIN HAT Template:PinHeader_2x20_P2.54mm_Vertical, symbol Connector:Raspberry_Pi_2_3
- added J1: Raspberry_Pi_2_3, FIN HAT Template:PinSocket_2x20_P2.54mm_Vertical, symbol FIN_HAT_TEMPLATE:Raspberry_Pi_2_3
- J2: footprint FIN HAT Template:PinHeader_2x02_P2.54mm_Vertical -> FIN HAT Template:PinSocket_2x02_P2.54mm_Vertical
- J3: footprint FIN HAT Template:PinHeader_2x09_P2.54mm_Vertical -> FIN HAT Template:PinSocket_2x09_P2.54mm_Vertical
- J4: footprint FIN HAT Template:PinHeader_1x04_P2.54mm_Vertical -> FIN HAT Template:PinSocket_1x04_P2.54mm_Vertical
Connections:
- net +3V3: now also J1.1 (3V3), J1.17 (3V3)
- net +5V: now also J1.2 (5V), J1.4 (5V)
- net GND: now also J1.14 (GND), J1.20 (GND), J1.25 (GND), J1.30 (GND), J1.34 (GND), J1.39 (GND), J1.6 (GND), J1.9 (GND)
Other:
- note removed: "USB Header"
Changed lines of the file:
@@
-	1    0    0    -1
-$EndComp
-$Comp
-L Connector:Raspberry_Pi_2_3 J1
-U 1 1 5F07B77A
-P 3550 3800
-F 0 "J1" H 2550 5200 50  0000 C CNN
-F 1 "Raspberry_Pi_2_3" H 2850 5100 50  0000 C CNN
-F 2 "FIN HAT Template:PinHeader_2x20_P2.54mm_Vertical" H 3550 3800 50  0001 C CNN
-F 3 "https://www.raspberrypi.org/documentation/hardware/raspberrypi/schematics/rpi_SCH_3bplus_1p0_reduced.pdf" H 3550 3800 50  0001 C CNN
-	1    3550 3800
 	1    0    0    -1
 $EndComp
@@
 Text Notes 7900 2550 0    50   ~ 0
 POE Header
-Text Notes 10100 2700 0    50   ~ 0
-USB Header
 Text Notes 4000 5100 0    50   ~ 0
 Raspberry Pi CM3 HAT Socket
@@
 Wire Wire Line
 	6700 1300 6700 1100
-$Comp
-L FIN_HAT_TEMPLATE:Co-Processor_Header J3
-U 1 1 5F1CE898
-P 9700 4050
-F 0 "J3" H 10050 4275 50  0000 C CNN
-F 1 "Co-Processor_Header" H 10050 4184 50  0000 C CNN
-F 2 "FIN HAT Template:PinHeader_2x09_P2.54mm_Vertical" H 9700 3650 50  0001 C CNN
-F 3 "~" H 9700 3650 50  0001 C CNN
-	1    9700 4050
-	1    0    0    -1
-$EndComp
 NoConn ~ 10600 4050
 $Comp
@@
 	9400 4850 9500 4850
 $Comp
-L FIN_HAT_TEMPLATE:POE_Header J2
-U 1 1 5F1D361B
-P 7900 2300
-F 0 "J2" H 8150 2525 50  0000 C CNN
-F 1 "POE_Header" H 8150 2434 50  0000 C CNN
-F 2 "FIN HAT Template:PinHeader_2x02_P2.54mm_Vertical" H 7900 2300 50  0001 C CNN
-F 3 "~" H 7900 2300 50  0001 C CNN
-	1    7900 2300
-	1    0    0    -1
-$EndComp
-$Comp
-L FIN_HAT_TEMPLATE:USB_Header J4
-U 1 1 5F1D6217
-P 10100 2300
-F 0 "J4" H 10328 2301 50  0000 L CNN
-F 1 "USB_Header" H 10328 2210 50  0000 L CNN
-F 2 "FIN HAT Template:PinHeader_1x04_P2.54mm_Vertical" H 10100 2300 50  0001 C CNN
-F 3 "~" H 10100 2300 50  0001 C CNN
-	1    10100 2300
-	1    0    0    -1
-$EndComp
-$Comp
 L power:GND #PWR09
 U 1 1 5F1D6ACD
@@
 Wire Wire Line
 	9800 2500 9800 2600
+$Comp
+L FIN_HAT_TEMPLATE:Raspberry_Pi_2_3 J1
+U 1 1 5F15F5E4
+P 3550 3800
+F 0 "J1" H 2550 5200 50  0000 C CNN
+F 1 "Raspberry_Pi_2_3" H 2850 5100 50  0000 C CNN
+F 2 "FIN HAT Template:PinSocket_2x20_P2.54mm_Vertical" H 3550 3800 50  0001 C CNN
+F 3 "https://www.raspberrypi.org/documentation/hardware/raspberrypi/schematics/rpi_SCH_3bplus_1p0_reduced.pdf" H 3550 3800 50  0001 C CNN
+	1    3550 3800
+	1    0    0    -1
+$EndComp
+$Comp
+L FIN_HAT_TEMPLATE:POE_Header J2
+U 1 1 5F162702
+P 7900 2300
+F 0 "J2" H 8150 2525 50  0000 C CNN
+F 1 "POE_Header" H 8150 2434 50  0000 C CNN
+F 2 "FIN HAT Template:PinSocket_2x02_P2.54mm_Vertical" H 7900 2300 50  0001 C CNN
+F 3 "~" H 7900 2300 50  0001 C CNN
+	1    7900 2300
+	1    0    0    -1
+$EndComp
+$Comp
+L FIN_HAT_TEMPLATE:Co-Processor_Header J3
+U 1 1 5F163428
+P 9700 4050
+F 0 "J3" H 10050 4275 50  0000 C CNN
+F 1 "Co-Processor_Header" H 10050 4184 50  0000 C CNN
+F 2 "FIN HAT Template:PinSocket_2x09_P2.54mm_Vertical" H 10050 4183 50  0001 C CNN
+F 3 "~" H 9700 3650 50  0001 C CNN
+	1    9700 4050
+	1    0    0    -1
+$EndComp
+$Comp
+L FIN_HAT_TEMPLATE:USB_Header J4
+U 1 1 5F165BD8
+P 10100 2300
+F 0 "J4" H 10328 2301 50  0000 L CNN
+F 1 "USB_Header" H 10328 2210 50  0000 L CNN
+F 2 "FIN HAT Template:PinSocket_1x04_P2.54mm_Vertical" H 10100 2300 50  0001 C CNN
+F 3 "~" H 10100 2300 50  0001 C CNN
+	1    10100 2300
+	1    0    0    -1
+$EndComp
 $EndSCHEMATC
